Commit message: continued work. Minimally working

File: framefab_robot/asw_end_effector/urdf/asw_eef_macro.xacro (robot description, xacro)
@@ -19,5 +19,6 @@
       <collision>
         <geometry>
-          <mesh filename="package://asw_end_effector/meshes/collision/asw_hotend_end_effector_hull.stl" scale=".001 .001 .001"/>
+          <!-- <mesh filename="package://asw_end_effector/meshes/collision/asw_hotend_end_effector_hull.stl" scale=".001 .001 .001"/> -->
+        <mesh filename="package://asw_end_effector/meshes/visual/asw_hotend_end_effector2.stl" scale=".001 .001 .001"/>
         </geometry>
         <material name="red">
@@ -41,5 +42,5 @@
         <parent link="${prefix}tmp_tcp_frame"/>
         <child link="${prefix}tcp_frame"/>
-        <origin xyz="0 0 0.002"/>
+        <origin xyz="0 0 0.001"/>
     </joint>
   </xacro:macro>

Commit message: Fixup

File: framefab_robot/asw_end_effector/urdf/asw_eef_macro.xacro (robot description, xacro)
@@ -42,5 +42,5 @@
         <parent link="${prefix}tmp_tcp_frame"/>
         <child link="${prefix}tcp_frame"/>
-        <origin xyz="0 0 0.001"/>
+        <origin xyz="0 0 0.0004"/>
     </joint>
   </xacro:macro>
